File: logboi.kicad_pcb (KiCad board)
At the start: 2 copper layers, 373.9 x 85.7 mm, 161 parts, among them J2 Conn_02x03_Odd_Even, K0 KEYSW, K1 KEYSW, K10 KEYSW, K11 KEYSW, K12 KEYSW, K13 KEYSW, K14 KEYSW, K15 KEYSW, K16 KEYSW, K17 KEYSW, K18 KEYSW, K19 KEYSW, K2 KEYSW, K20 KEYSW, K21 KEYSW, K22 KEYSW, K23 KEYSW, K24 KEYSW, K25 KEYSW, K26 KEYSW, K27 KEYSW, K28 KEYSW, K29 KEYSW, K3 KEYSW, K30 KEYSW, K31 KEYSW, K32 KEYSW, K33 KEYSW, K34 KEYSW, K35 KEYSW, K36 KEYSW, K37 KEYSW, K38 KEYSW, K39 KEYSW, K4 KEYSW, K40 KEYSW, K41 KEYSW, K42 KEYSW, K43 KEYSW, K44 KEYSW, K45 KEYSW, K46 KEYSW, K47 KEYSW, K48 KEYSW, K49 KEYSW, K5 KEYSW, K50 KEYSW, K51 KEYSW, K52 KEYSW, K53 KEYSW, K54 KEYSW, K55 KEYSW, K56 KEYSW, K57 KEYSW, K58 KEYSW, K59 KEYSW, K6 KEYSW, K60 KEYSW, K61 KEYSW, K62 KEYSW, K63 KEYSW, K64 KEYSW, K65 KEYSW, K66 KEYSW, K67 KEYSW, K68 KEYSW, K69 KEYSW, K7 KEYSW, K8 KEYSW, K9 KEYSW, P1 USB_C_Plug_USB2.0, SW1 Reset_SW, U1 ATmega32U4-AU, Y1 Crystal

Commit message: Add files via upload
Parts:
- K56: footprint Button_Switch_Keyboard:SW_Cherry_MX_1.00u_PCB -> Button_Switch_Keyboard:SW_Cherry_MX_1.25u_PCB
- moved K2 2.38 mm to (77.8, 24.8)
- moved K20 2.38 mm to (77.8, 43.8)
- moved K21 2.38 mm to (96.9, 43.8)
- moved K22 2.38 mm to (120.7, 43.8)
- moved K3 2.38 mm to (96.9, 24.8)
- moved K37 2.38 mm to (77.8, 62.9)
- moved K38 2.38 mm to (96.9, 62.9)
- moved K39 2.38 mm to (125.5, 62.9)
- moved K53 2.38 mm to (77.8, 81.9)
- moved K54 2.38 mm to (96.9, 81.9)
- moved D1 2.38 mm to (52.4, 33.7)
- moved D19 2.38 mm to (52.4, 52.7)
- moved D36 2.38 mm to (52.4, 71.8)
- moved D52 2.38 mm to (42.9, 90.8)
- moved K0 2.38 mm to (39.7, 24.8)
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Routing:
- net /Col_4: track 142.2 -> 147.1 mm
- net /Row_1: track 500.4 -> 505.2 mm
- net /Row_2: track 636.0 -> 639.3 mm
- net /Col_1: track 228.6 -> 231.3 mm
- net /Col_3: track 178.2 -> 180.6 mm
- net /Col_2: track 206.3 -> 208.6 mm
- net /Col_0: track 249.7 -> 252.1 mm
- net /Row_0: track 604.9 -> 607.3 mm
Other:
- board size 373.9 x 85.7 mm -> 376.2 x 85.7 mm

Commit message: Add files via upload
Parts:
- removed C1: 0.1u, Capacitor_SMD:C_0805_2012Metric_Pad1.15x1.40mm_HandSolder
- added F1: Polyfuse, Fuse:Fuse_1206_3216Metric, B.Cu at (355.2, 34.6)
- added R5: 5.1k, Resistor_SMD:R_0805_2012Metric_Pad1.15x1.40mm_HandSolder, B.Cu at (345.5, 23.2)
- added R6: 5.1k, Resistor_SMD:R_0805_2012Metric_Pad1.15x1.40mm_HandSolder, B.Cu at (363.8, 22.7)
- C5: value 4.7u -> 10u
- D0, D1, D10, D11, D12, D13, D14, D15, D16, D17, D18, D19, D2, D20, D21, D22, D23, D24, D25, D26, D27, D28, D29, D3, D30, D31, D32, D33, D34, D35, D36, D37, D38, D39, D4, D40, D41, D42, D43, D44, D45, D46, D47, D48, D49, D5, D50, D51, D52, D53, D54, D55, D56, D57, D58, D59, D6, D60, D61, D62, D63, D64, D65, D66, D67, D68, D69, D7, D8, D9: footprint Diode_SMD:D_0805_2012Metric_Pad1.15x1.40mm_HandSolder -> Diode_SMD:D_SOD-323F
- H1, H2, H3, H4: footprint MountingHole:MountingHole_3.2mm_M3_DIN965 -> random-keyboard-parts:M2 Mounting Hole
- P1: footprint Connector_USB:USB_C_Receptacle_Amphenol_12401610E4-2A_CircularHoles -> Type-C:USB_C_GCT_USB4085
- SW1: footprint Button_Switch_SMD:SW_Push_1P1T_NO_6x6mm_H9.5mm -> random-keyboard-parts:SKQG-1155865
- U1: footprint Package_QFP:TQFP-44_10x10mm_P0.8mm -> Package_DFN_QFN:QFN-48-1EP_7x7mm_P0.5mm_EP5.6x5.6mm
- Y1: footprint Crystal:Crystal_SMD_5032-2Pin_5.0x3.2mm_HandSoldering -> Crystal:Crystal_SMD_3225-4Pin_3.2x2.5mm
- moved C4 180.7 mm to (168.1, 91.4), turned to 270 degrees
- moved C2 177.7 mm to (180.8, 97.3), turned to 270 degrees
- moved C3 175.4 mm to (172.3, 78.8), turned to 0 degrees
- moved C5 168.2 mm to (181.3, 77.8), turned to 180 degrees
- moved J2 89.8 mm to (150.7, 88.6)
- moved C7 27.0 mm to (176.3, 98.1)
- moved R2 24.1 mm to (355.8, 29.3), turned to 90 degrees
- moved Y1 23.5 mm to (170.4, 98.1), turned to 0 degrees
- moved R3 23.1 mm to (357.7, 29.3), turned to 90 degrees
- moved C6 14.6 mm to (164.4, 98.0), turned to 270 degrees
- moved R4 3.42 mm to (169.3, 80.4)
- moved P1 3.16 mm to (356.3, 18.2)
- moved C8 1.86 mm to (186.8, 87.4), turned to 0 degrees
- moved U1 0.42 mm to (177.3, 86.9)
- moved D62 0.13 mm to (304.9, 90.7)
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Connections:
- P1 pad A4: VCC -> Net-(F1-Pad2)
- P1 pad A8: (no net) -> Net-(P1-PadA8)
- P1 pad A9: VCC -> Net-(F1-Pad2)
- P1 pad B4: VCC -> Net-(F1-Pad2)
- P1 pad B6: (no net) -> Net-(P1-PadA6)
- P1 pad B7: (no net) -> Net-(P1-PadA7)
- P1 pad B8: (no net) -> Net-(P1-PadB8)
- P1 pad B9: VCC -> Net-(F1-Pad2)
- U1 pad 10: /Row_3 -> /Col_16
- U1 pad 11: /Row_2 -> /Col_17
- U1 pad 12: /Row_1 -> /Row_5
- U1 pad 18: /Row_0 -> /Row_4
- U1 pad 19: /Col_17 -> /Row_0
- U1 pad 20: /Col_16 -> /Row_1
- U1 pad 21: /Col_15 -> /Row_2
- U1 pad 22: /Col_14 -> /Row_3
- U1 pad 25: /Col_7 -> /Col_0
- U1 pad 26: /Col_6 -> /Col_1
- U1 pad 27: /Col_5 -> /Col_2
- U1 pad 28: /Col_4 -> /Col_3
- U1 pad 29: /Col_3 -> /Col_4
- U1 pad 30: /Col_2 -> /Col_5
- U1 pad 31: /Col_1 -> /Col_6
- U1 pad 32: /Col_0 -> /Col_7
- U1 pad 8: /Row_5 -> /Col_14
- U1 pad 9: /Row_4 -> /Col_15
- Y1 pad 2: Net-(C7-Pad1) -> GND
Routing:
- net /Row_3: track 527.3 -> 402.8 mm, vias 32 -> 29
- net /Row_0: track 607.3 -> 517.0 mm
- net /Col_0: track 252.1 -> 199.3 mm
- net /Row_2: track 639.3 -> 592.0 mm, vias 36 -> 37
- net VCC: track 373.5 -> 327.0 mm, vias 4 -> 7
- net /Col_2: track 208.6 -> 174.5 mm, vias 6 -> 5
- net /Col_7: track 171.9 -> 138.0 mm, vias 8 -> 7
- net Net-(C7-Pad1): track 45.6 -> 13.5 mm
- net /Col_1: track 231.3 -> 199.9 mm, vias 6 -> 7
- net GND: track 384.7 -> 414.0 mm, vias 4 -> 8
- net /Col_6: track 133.5 -> 107.5 mm, vias 6 -> 5
- net /Row_1: track 505.2 -> 529.2 mm
- net Net-(P1-PadA7): track 29.1 -> 6.11 mm
- net /Col_3: track 180.6 -> 159.6 mm, vias 6 -> 5
- net Net-(P1-PadA6): track 26.2 -> 6.49 mm, vias 0 -> 1
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- added copper zone on B.Cu, net GND
- added copper zone on F.Cu, net GND
Other:
- board text added: ".len()"

Commit message: Add files via upload
Parts:
- K17, K51: footprint Button_Switch_Keyboard:SW_Cherry_MX_1.00u_PCB -> Button_Switch_Keyboard:SW_Cherry_MX_1.50u_PCB
- K34: footprint Button_Switch_Keyboard:SW_Cherry_MX_1.75u_PCB -> Button_Switch_Keyboard:SW_Cherry_MX_2.25u_PCB
- K60: footprint Button_Switch_Keyboard:SW_Cherry_MX_2.25u_PCB -> Button_Switch_Keyboard:SW_Cherry_MX_2.75u_PCB
- moved C2 7.14 mm to (173.6, 97.3)
- moved C3 7.14 mm to (165.1, 78.8)
- moved C6 7.14 mm to (157.2, 98.0)
- moved C7 7.14 mm to (169.1, 98.1)
- moved D10 7.14 mm to (221.5, 33.6)
- moved D12 7.14 mm to (259.6, 33.6)
- moved D13 7.14 mm to (278.6, 33.6)
- moved D15 7.14 mm to (316.7, 33.6)
- moved D16 7.14 mm to (335.8, 33.6)
- moved D23 7.14 mm to (131.0, 52.6)
- moved D24 7.14 mm to (150.1, 52.6)
- moved D26 7.14 mm to (188.2, 52.6)
- moved D28 7.14 mm to (226.3, 52.6)
- moved D29 7.14 mm to (245.3, 52.6)
- moved D30 7.14 mm to (264.4, 52.6)
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Routing:
- net /Row_3: track 402.8 -> 419.3 mm
- net /Col_16: track 297.5 -> 311.4 mm
- net /Col_17: track 300.8 -> 314.3 mm
- net /Col_12: track 256.7 -> 266.7 mm
- net /Col_9: track 201.6 -> 211.5 mm
- net /Row_1: track 529.2 -> 539.0 mm
- net /Col_13: track 275.2 -> 284.7 mm
- net /Col_10: track 219.9 -> 229.4 mm
- net /Col_11: track 238.3 -> 247.8 mm
- net /Row_2: track 592.0 -> 599.4 mm
- net /Col_14: track 226.7 -> 232.1 mm
- net /Col_8: track 171.9 -> 176.7 mm
- net /Row_0: track 517.0 -> 521.8 mm
Other:
- board size 376.2 x 85.7 mm -> 385.8 x 85.7 mm

Commit message: Add files via upload
Parts:
- K22: footprint Button_Switch_Keyboard:SW_Cherry_MX_1.50u_PCB -> Button_Switch_Keyboard:SW_Cherry_MX_1.75u_PCB
- K39: footprint Button_Switch_Keyboard:SW_Cherry_MX_2.00u_PCB -> Button_Switch_Keyboard:SW_Cherry_MX_2.25u_PCB
- K4, K55: footprint Button_Switch_Keyboard:SW_Cherry_MX_1.25u_PCB -> Button_Switch_Keyboard:SW_Cherry_MX_1.50u_PCB
- K50: footprint Button_Switch_Keyboard:SW_Cherry_MX_1.25u_PCB -> Button_Switch_Keyboard:SW_Cherry_MX_1.75u_PCB
- K51: footprint Button_Switch_Keyboard:SW_Cherry_MX_1.50u_PCB -> Button_Switch_Keyboard:SW_Cherry_MX_1.00u_Plate
- moved D2 4.76 mm to (59.6, 33.6)
- moved D1 4.76 mm to (40.5, 33.6)
- moved D20 4.76 mm to (59.5, 52.6)
- moved D21 4.76 mm to (78.6, 52.6)
- moved D3 4.76 mm to (78.6, 33.6)
- moved D36 4.76 mm to (40.5, 71.7)
- moved H2 4.76 mm to (53.9, 77.5)
- moved H3 4.76 mm to (53.9, 39.4)
- moved K2 4.76 mm to (65.9, 24.8)
- moved K20 4.76 mm to (65.9, 43.8)
- moved K21 4.76 mm to (85.0, 43.8)
- moved K3 4.76 mm to (85.0, 24.8)
- moved K37 4.76 mm to (65.9, 62.9)
- moved K38 4.76 mm to (85.0, 62.9)
- moved K53 4.76 mm to (65.9, 81.9)
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Routing:
- net /Row_2: track 599.4 -> 611.0 mm
- net /Col_15: track 251.2 -> 260.8 mm
- net /Col_16: track 311.4 -> 321.0 mm
- net /Row_0: track 521.8 -> 531.3 mm
- net /Row_1: track 539.0 -> 548.4 mm
- net /Col_3: track 159.6 -> 165.7 mm
- net /Col_1: track 199.9 -> 204.9 mm
- net /Col_0: track 199.3 -> 204.1 mm
- net /Col_2: track 174.5 -> 179.2 mm
- net /Row_3: track 419.3 -> 423.9 mm
- net /Col_4: track 128.5 -> 132.2 mm
- net Net-(C6-Pad1): track 24.7 -> 22.4 mm
- net VCC: track 327.0 -> 325.8 mm
- net /Col_12: track 266.7 -> 267.7 mm
- net GND: track 414.0 -> 414.5 mm
Other:
- board size 385.8 x 85.7 mm -> 390.5 x 85.7 mm
- rule trace_min: 0.2 -> 0

Commit message: Add files via upload
Parts:
- moved J2 88.0 mm to (231.5, 91.6), turned to 270 degrees
Connections:
- J2 pad 2: /Row_2 -> /Col_17
- J2 pad 3: /Row_4 -> /Col_16
- J2 pad 4: /Row_3 -> /Col_15
Routing:
- net /Row_4: track 45.4 -> 0.00 mm, vias 1 -> 0
- net VCC: track 325.8 -> 345.0 mm, vias 7 -> 8
- net GND: track 414.5 -> 430.6 mm, vias 8 -> 9
- net /Row_3: track 423.9 -> 412.0 mm
- net /Col_16: track 321.0 -> 328.6 mm, vias 5 -> 6
- net /Row_2: track 611.0 -> 605.6 mm, vias 37 -> 36
- net /Col_17: track 314.7 -> 320.0 mm, vias 5 -> 6
- net /Col_15: track 260.8 -> 265.1 mm, vias 5 -> 6
- net /Reset: track 81.9 -> 85.6 mm, vias 2 -> 3
- net /Col_14: track 232.1 -> 233.6 mm
