File: Longboi/longboi.kicad_pcb (KiCad board)
At the start: 2 copper layers, 390.5 x 85.7 mm, 163 parts, among them J2 Conn_02x03_Odd_Even, K0 KEYSW, K1 KEYSW, K10 KEYSW, K11 KEYSW, K12 KEYSW, K13 KEYSW, K14 KEYSW, K15 KEYSW, K16 KEYSW, K17 KEYSW, K18 KEYSW, K19 KEYSW, K2 KEYSW, K20 KEYSW, K21 KEYSW, K22 KEYSW, K23 KEYSW, K24 KEYSW, K25 KEYSW, K26 KEYSW, K27 KEYSW, K28 KEYSW, K29 KEYSW, K3 KEYSW, K30 KEYSW, K31 KEYSW, K32 KEYSW, K33 KEYSW, K34 KEYSW, K35 KEYSW, K36 KEYSW, K37 KEYSW, K38 KEYSW, K39 KEYSW, K4 KEYSW, K40 KEYSW, K41 KEYSW, K42 KEYSW, K43 KEYSW, K44 KEYSW, K45 KEYSW, K46 KEYSW, K47 KEYSW, K48 KEYSW, K49 KEYSW, K5 KEYSW, K50 KEYSW, K51 KEYSW, K52 KEYSW, K53 KEYSW, K54 KEYSW, K55 KEYSW, K56 KEYSW, K57 KEYSW, K58 KEYSW, K59 KEYSW, K6 KEYSW, K60 KEYSW, K61 KEYSW, K62 KEYSW, K63 KEYSW, K64 KEYSW, K65 KEYSW, K66 KEYSW, K67 KEYSW, K68 KEYSW, K69 KEYSW, K7 KEYSW, K8 KEYSW, K9 KEYSW, P1 USB_C_Plug_USB2.0, SW1 Reset_SW, U1 ATmega32U4-AU, Y1 Crystal

Commit message: update LongBoi for second prototype
update LongBoi for second prototype
Parts:
- removed Y1: Crystal, Crystal:Crystal_SMD_3225-4Pin_3.2x2.5mm
- added C1: Crystal, Crystal:Crystal_SMD_3225-4Pin_3.2x2.5mm, B.Cu at (328.4, 68.5)
- added G1: dotlen, Images:dotlen_14, F.Cu at (202.5, 87.0)
- added G2: string_dotlen, Images:string-dotlen_90mm_high, B.Cu at (200.3, 70.4)
- added G3: string, Images:String_5.7mm_high, F.Cu at (170.4, 87.8)
- added H5: MountingHole, random-keyboard-parts:M2 Mounting Hole, F.Cu at (211.0, 58.4)
- added K22-spacer1: KEYSW, MX_Only:MXOnly-1.25U-NoLED, F.Cu at (113.4, 48.9)
- added K22-stepped1: KEYSW, MX_Only:MXOnly-1.25U-NoLED, F.Cu at (103.9, 48.9)
- added K3-2uVert1: KEYSW, MX_Only:MXOnly-2U-NoLED, F.Cu at (82.4, 39.4)
- added K38-2uVert1: KEYSW, MX_Only:MXOnly-2U-NoLED, F.Cu at (82.4, 77.5)
- added K39-spacer1: KEYSW, MX_Only:MXOnly-1.75U-NoLED, F.Cu at (118.2, 67.9)
- added K4-spacer1: KEYSW, MX_Only:MXOnly-1U-NoLED, F.Cu at (111.0, 29.8)
- added K52-1u1: KEYSW, MX_Only:MXOnly-1U-NoLED, F.Cu at (25.3, 87.0)
- added K52-2u1: KEYSW, MX_Only:MXOnly-2U-ReversedStabilizers-NoLED, F.Cu at (53.9, 87.0)
- added K55-1.25: KEYSW, MX_Only:MXOnly-1.25U-NoLED, F.Cu at (103.9, 87.0)
- added K55-spacer1: KEYSW, MX_Only:MXOnly-1.25U-NoLED, F.Cu at (113.4, 87.0)
- added K56-1.25: KEYSW, MX_Only:MXOnly-1.25U-NoLED, F.Cu at (127.7, 87.0)
- added K57-1.25: KEYSW, MX_Only:MXOnly-1.25U-NoLED, F.Cu at (151.5, 87.0)
- added K57-1.5u1: KEYSW, MX_Only:MXOnly-1.5U-NoLED, F.Cu at (134.8, 87.0)
- added K57-1u1: KEYSW, MX_Only:MXOnly-1U-NoLED, F.Cu at (153.9, 87.0)
- added K58-6u1: KEYSW, MX_Only:MXOnly-6.25U-ReversedStabilizers-NoLED, F.Cu at (222.9, 87.0)
- added K58for1.25Row1: KEYSW, MX_Only:MXOnly-2.25U-ReversedStabilizers-NoLED, F.Cu at (184.8, 87.0)
- added K59-1.25u1: KEYSW, MX_Only:MXOnly-1.25U-NoLED, F.Cu at (218.2, 87.0)
- added K59-7u1: KEYSW, MX_Only:MXOnly-7U-ReversedStabilizers-NoLED, F.Cu at (215.8, 87.0)
- added K59Alt1: KEYSW, MX_Only:MXOnly-2.75U-ReversedStabilizers-NoLED, F.Cu at (237.2, 87.0)
- added K60Alt1: KEYSW, MX_Only:MXOnly-1U-NoLED, F.Cu at (272.9, 87.0)
- added K61-1.5u1: KEYSW, MX_Only:MXOnly-1.5U-NoLED, F.Cu at (296.7, 87.0)
- added K62-1.5u1: KEYSW, MX_Only:MXOnly-1.5U-NoLED, F.Cu at (325.3, 87.0)
- added SW3: Rotary_Encoder_Switch, random-keyboard-parts:RotaryEncoder_Alps_EC11E-Switch_Vertical_H20mm_MX-1U, F.Cu at (387.2, 29.8)
- D0, D1, D10, D11, D12, D13, D14, D15, D16, D17, D18, D19, D2, D20, D21, D22, D23, D24, D25, D26, D27, D28, D29, D3, D30, D31, D32, D33, D34, D35, D36, D37, D38, D39, D4, D40, D41, D42, D43, D44, D45, D46, D47, D48, D49, D5, D50, D51, D52, D53, D54, D55, D56, D57, D58, D59, D6, D60, D61, D62, D63, D64, D65, D66, D67, D68, D69, D7, D8, D9: value D -> SOD-323F
- F1: value Polyfuse -> 500mA
- J2: value Conn_02x03_Odd_Even -> ICSP_Header
- K0, K1, K10, K11, K12, K13, K14, K15, K16, K18, K19, K2, K20, K21, K23, K24, K25, K26, K27, K28, K29, K3, K30, K31, K32, K33, K35, K36, K37, K38, K40, K41, K42, K43, K44, K45, K46, K47, K48, K49, K5, K53, K54, K59, K6, K61, K62, K63, K64, K65, K66, K67, K68, K69, K7, K8, K9: footprint Button_Switch_Keyboard:SW_Cherry_MX_1.00u_PCB -> MX_Only:MXOnly-1U-NoLED
- K17, K4, K55: footprint Button_Switch_Keyboard:SW_Cherry_MX_1.50u_PCB -> MX_Only:MXOnly-1.5U-NoLED
- K22, K50: footprint Button_Switch_Keyboard:SW_Cherry_MX_1.75u_PCB -> MX_Only:MXOnly-1.75U-NoLED
- K34, K39, K58: footprint Button_Switch_Keyboard:SW_Cherry_MX_2.25u_PCB -> MX_Only:MXOnly-2.25U-ReversedStabilizers-NoLED
- K51: footprint Button_Switch_Keyboard:SW_Cherry_MX_1.00u_Plate -> MX_Only:MXOnly-1U-NoLED
- K52: footprint Button_Switch_Keyboard:SW_Cherry_MX_2.00u_PCB -> MX_Only:MXOnly-2U-ReversedStabilizers-NoLED
- K56, K57: footprint Button_Switch_Keyboard:SW_Cherry_MX_1.25u_PCB -> MX_Only:MXOnly-1.25U-NoLED
- K60: footprint Button_Switch_Keyboard:SW_Cherry_MX_2.75u_PCB -> MX_Only:MXOnly-2.75U-ReversedStabilizers-NoLED
- P1: value USB_C_Plug_USB2.0 -> 918-418K2023S40001; footprint Type-C:USB_C_GCT_USB4085 -> Connector_USB:918-418K2023S40001
- SW1: value Reset_SW -> Reset_Switch
- U1: value ATmega32U4-AU -> ATmega32U4-MUR
- moved C7 167.6 mm to (331.9, 68.6)
- moved C6 167.6 mm to (325.1, 68.5)
- moved C4 165.0 mm to (323.3, 61.6), turned to 0 degrees
- moved R4 162.2 mm to (322.1, 53.8)
- moved U1 161.7 mm to (329.3, 58.4)
- moved C2 161.4 mm to (331.7, 64.8), turned to 180 degrees
- moved C3 160.9 mm to (324.1, 53.8), turned to 90 degrees
- moved C8 160.5 mm to (337.4, 57.4), turned to 180 degrees
- moved C5 160.3 mm to (332.4, 52.0), turned to 90 degrees
- moved R1 153.6 mm to (348.9, 59.8), turned to 90 degrees
- moved SW1 152.6 mm to (355.0, 60.1)
- moved J2 123.0 mm to (351.7, 65.5)
- moved H1 57.2 mm to (320.6, 39.4)
- moved H4 57.2 mm to (320.6, 77.5)
- moved H2 38.1 mm to (92.0, 77.5)
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Connections:
- D38 pad 2: Net-(D38-Pad2) -> /Col_3
- K0 pad 1: /Col_0 -> Net-(D0-Pad2)
- K0 pad 2: Net-(D0-Pad2) -> /Col_0
- K1 pad 1: /Col_1 -> Net-(D1-Pad2)
- K1 pad 2: Net-(D1-Pad2) -> /Col_1
- K10 pad 1: /Col_10 -> Net-(D10-Pad2)
- K10 pad 2: Net-(D10-Pad2) -> /Col_10
- K11 pad 1: /Col_11 -> Net-(D11-Pad2)
- K11 pad 2: Net-(D11-Pad2) -> /Col_11
- K12 pad 1: /Col_12 -> Net-(D12-Pad2)
- K12 pad 2: Net-(D12-Pad2) -> /Col_12
- K13 pad 1: /Col_13 -> Net-(D13-Pad2)
- K13 pad 2: Net-(D13-Pad2) -> /Col_13
- K14 pad 1: /Col_14 -> Net-(D14-Pad2)
- K14 pad 2: Net-(D14-Pad2) -> /Col_14
- K15 pad 1: /Col_15 -> Net-(D15-Pad2)
- K15 pad 2: Net-(D15-Pad2) -> /Col_15
- K16 pad 1: /Col_16 -> Net-(D16-Pad2)
- K16 pad 2: Net-(D16-Pad2) -> /Col_16
- K17 pad 1: /Col_17 -> Net-(D17-Pad2)
- K17 pad 2: Net-(D17-Pad2) -> /Col_17
- K18 pad 1: /Col_0 -> Net-(D18-Pad2)
- K18 pad 2: Net-(D18-Pad2) -> /Col_0
- K19 pad 1: /Col_1 -> Net-(D19-Pad2)
- K19 pad 2: Net-(D19-Pad2) -> /Col_1
- K2 pad 1: /Col_2 -> Net-(D2-Pad2)
- K2 pad 2: Net-(D2-Pad2) -> /Col_2
- K20 pad 1: /Col_2 -> Net-(D20-Pad2)
- K20 pad 2: Net-(D20-Pad2) -> /Col_2
- K21 pad 1: /Col_3 -> Net-(D21-Pad2)
- K21 pad 2: Net-(D21-Pad2) -> /Col_3
- K22 pad 1: /Col_4 -> Net-(D22-Pad2)
- K22 pad 2: Net-(D22-Pad2) -> /Col_4
- K23 pad 1: /Col_5 -> Net-(D23-Pad2)
- K23 pad 2: Net-(D23-Pad2) -> /Col_5
- K24 pad 1: /Col_6 -> Net-(D24-Pad2)
- K24 pad 2: Net-(D24-Pad2) -> /Col_6
- K25 pad 1: /Col_7 -> Net-(D25-Pad2)
- K25 pad 2: Net-(D25-Pad2) -> /Col_7
- K26 pad 1: /Col_8 -> Net-(D26-Pad2)
- K26 pad 2: Net-(D26-Pad2) -> /Col_8
- K27 pad 1: /Col_9 -> Net-(D27-Pad2)
- K27 pad 2: Net-(D27-Pad2) -> /Col_9
- K28 pad 1: /Col_10 -> Net-(D28-Pad2)
- K28 pad 2: Net-(D28-Pad2) -> /Col_10
- K29 pad 1: /Col_11 -> Net-(D29-Pad2)
- K29 pad 2: Net-(D29-Pad2) -> /Col_11
- K3 pad 1: /Col_3 -> Net-(D3-Pad2)
- K3 pad 2: Net-(D3-Pad2) -> /Col_3
- K30 pad 1: /Col_12 -> Net-(D30-Pad2)
- K30 pad 2: Net-(D30-Pad2) -> /Col_12
- K31 pad 1: /Col_13 -> Net-(D31-Pad2)
- K31 pad 2: Net-(D31-Pad2) -> /Col_13
- K32 pad 1: /Col_14 -> Net-(D32-Pad2)
- K32 pad 2: Net-(D32-Pad2) -> /Col_14
- K33 pad 1: /Col_15 -> Net-(D33-Pad2)
- K33 pad 2: Net-(D33-Pad2) -> /Col_15
- K34 pad 1: /Col_16 -> Net-(D34-Pad2)
- K34 pad 2: Net-(D34-Pad2) -> /Col_16
- K35 pad 1: /Col_0 -> Net-(D35-Pad2)
- K35 pad 2: Net-(D35-Pad2) -> /Col_0
- K36 pad 1: /Col_1 -> Net-(D36-Pad2)
- K36 pad 2: Net-(D36-Pad2) -> /Col_1
- K37 pad 1: /Col_2 -> Net-(D37-Pad2)
- K37 pad 2: Net-(D37-Pad2) -> /Col_2
- K38 pad 2: Net-(D38-Pad2) -> Net-(K38-2uVert1-Pad2)
- K39 pad 1: /Col_4 -> Net-(D39-Pad2)
- K39 pad 2: Net-(D39-Pad2) -> /Col_4
- K4 pad 1: /Col_4 -> Net-(D4-Pad2)
- K4 pad 2: Net-(D4-Pad2) -> /Col_4
- K40 pad 1: /Col_5 -> Net-(D40-Pad2)
- K40 pad 2: Net-(D40-Pad2) -> /Col_5
- K41 pad 1: /Col_6 -> Net-(D41-Pad2)
- K41 pad 2: Net-(D41-Pad2) -> /Col_6
- K42 pad 1: /Col_7 -> Net-(D42-Pad2)
- K42 pad 2: Net-(D42-Pad2) -> /Col_7
- K43 pad 1: /Col_8 -> Net-(D43-Pad2)
- K43 pad 2: Net-(D43-Pad2) -> /Col_8
- K44 pad 1: /Col_9 -> Net-(D44-Pad2)
- K44 pad 2: Net-(D44-Pad2) -> /Col_9
- K45 pad 1: /Col_10 -> Net-(D45-Pad2)
- K45 pad 2: Net-(D45-Pad2) -> /Col_10
- K46 pad 1: /Col_11 -> Net-(D46-Pad2)
- K46 pad 2: Net-(D46-Pad2) -> /Col_11
- K47 pad 1: /Col_12 -> Net-(D47-Pad2)
- K47 pad 2: Net-(D47-Pad2) -> /Col_12
- K48 pad 1: /Col_13 -> Net-(D48-Pad2)
- K48 pad 2: Net-(D48-Pad2) -> /Col_13
- K49 pad 1: /Col_14 -> Net-(D49-Pad2)
- K49 pad 2: Net-(D49-Pad2) -> /Col_14
- K5 pad 1: /Col_5 -> Net-(D5-Pad2)
- K5 pad 2: Net-(D5-Pad2) -> /Col_5
- K50 pad 1: /Col_15 -> Net-(D50-Pad2)
- K50 pad 2: Net-(D50-Pad2) -> /Col_15
- K51 pad 1: /Col_16 -> Net-(D51-Pad2)
- K51 pad 2: Net-(D51-Pad2) -> /Col_16
- K52 pad 1: /Col_0 -> Net-(D52-Pad2)
- K52 pad 2: Net-(D52-Pad2) -> /Col_0
- K53 pad 1: /Col_1 -> Net-(D53-Pad2)
- K53 pad 2: Net-(D53-Pad2) -> /Col_1
- K54 pad 1: /Col_2 -> Net-(D54-Pad2)
- K54 pad 2: Net-(D54-Pad2) -> /Col_2
- K55 pad 1: /Col_3 -> Net-(D55-Pad2)
- K55 pad 2: Net-(D55-Pad2) -> /Col_3
- K56 pad 1: /Col_4 -> Net-(D56-Pad2)
- K56 pad 2: Net-(D56-Pad2) -> /Col_4
- K57 pad 1: /Col_5 -> Net-(D57-Pad2)
- K57 pad 2: Net-(D57-Pad2) -> /Col_5
- K58 pad 1: /Col_6 -> Net-(D58-Pad2)
- K58 pad 2: Net-(D58-Pad2) -> /Col_7
- K59 pad 1: /Col_7 -> Net-(D59-Pad2)
- K59 pad 2: Net-(D59-Pad2) -> /Col_8
- K6 pad 1: /Col_6 -> Net-(D6-Pad2)
- K6 pad 2: Net-(D6-Pad2) -> /Col_6
- K60 pad 1: /Col_8 -> Net-(D60-Pad2)
- K60 pad 2: Net-(D60-Pad2) -> /Col_10
- K61 pad 1: /Col_9 -> Net-(D61-Pad2)
- K61 pad 2: Net-(D61-Pad2) -> /Col_11
- K62 pad 1: /Col_10 -> Net-(D62-Pad2)
- K62 pad 2: Net-(D62-Pad2) -> /Col_12
- K63 pad 1: /Col_11 -> Net-(D63-Pad2)
- K63 pad 2: Net-(D63-Pad2) -> /Col_13
- K64 pad 1: /Col_12 -> Net-(D64-Pad2)
- K64 pad 2: Net-(D64-Pad2) -> /Col_14
- K65 pad 1: /Col_13 -> Net-(D65-Pad2)
- K65 pad 2: Net-(D65-Pad2) -> /Col_15
- K66 pad 1: /Col_17 -> Net-(D66-Pad2)
- K66 pad 2: Net-(D66-Pad2) -> /Col_17
- K67 pad 1: /Col_17 -> Net-(D67-Pad2)
- K67 pad 2: Net-(D67-Pad2) -> /Col_17
- K68 pad 1: /Col_17 -> Net-(D68-Pad2)
- K68 pad 2: Net-(D68-Pad2) -> /Col_17
- K69 pad 1: /Col_16 -> Net-(D69-Pad2)
- K69 pad 2: Net-(D69-Pad2) -> /Col_16
- K7 pad 1: /Col_7 -> Net-(D7-Pad2)
- K7 pad 2: Net-(D7-Pad2) -> /Col_7
- K8 pad 1: /Col_8 -> Net-(D8-Pad2)
- K8 pad 2: Net-(D8-Pad2) -> /Col_8
- K9 pad 1: /Col_9 -> Net-(D9-Pad2)
- K9 pad 2: Net-(D9-Pad2) -> /Col_9
- P1 pad A8: Net-(P1-PadA8) -> unconnected-(P1-PadA8)
- P1 pad B8: Net-(P1-PadB8) -> unconnected-(P1-PadB8)
- U1 pad 1: /Row_6 -> Rotary_B
- U1 pad 12: /Row_5 -> Rotary_A
- U1 pad 18: /Row_4 -> /Row_3
- U1 pad 19: /Row_0 -> /Row_2
- U1 pad 21: /Row_2 -> /Row_0
- U1 pad 22: /Row_3 -> /Row_4
- U1 pad 42: Net-(U1-Pad42) -> unconnected-(U1-Pad42)
Routing:
- net VCC: track 350.9 -> 108.7 mm, vias 8 -> 6
- net GND: track 448.7 -> 207.7 mm, vias 8 -> 4
- net /Col_16: track 328.6 -> 134.1 mm, vias 6 -> 0
- net /Col_3: track 165.3 -> 347.6 mm, vias 5 -> 1
- net Net-(R2-Pad1): track 213.1 -> 32.0 mm
- net Net-(R3-Pad1): track 213.8 -> 32.8 mm
- net /Col_17: track 320.2 -> 142.6 mm, vias 6 -> 0
- net /Col_4: track 131.8 -> 307.3 mm, vias 5 -> 1
- net /Col_0: track 204.7 -> 368.4 mm, vias 6 -> 1
- net /Col_15: track 265.1 -> 101.6 mm, vias 6 -> 0
- net /Col_5: track 100.0 -> 258.8 mm, vias 6 -> 1
- net /Row_2: track 604.4 -> 448.2 mm, vias 36 -> 2
- net /Col_2: track 179.6 -> 332.4 mm, vias 5 -> 1
- net /Col_1: track 205.7 -> 353.6 mm, vias 7 -> 1
- net /Col_13: track 284.1 -> 151.5 mm, vias 6 -> 1
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- added copper zone on F.Cu, net Net-(D56-Pad2)
Other:
- board size 390.5 x 85.7 mm -> 383 x 78.2 mm
- net class Default removed
- board text added: "1.25u"
- board text added: "1.25u stepped"
- board text added: "1.5u"
- board text added: "1.75u"
- board text added: "1u"
- board text added: "2.25u"
- board text added: "2.75u"
- board text added: "2u"
- board text added: "2u Vertical"
- board text added: "6.25u"
- board text added: "7u"
- board text added: "7u-1.25u-1u-6.25u"
- board text added: "Optional EC11"
- board text added: "Stab Hole Pairings"
- board text added: "Supported Layouts"
- board text removed: ".len()"
