File: Longboi/longboi.kicad_sch (KiCad schematic)
At the start: 202 parts, among them J2 ICSP_Header, K0 KEYSW, K0-2uVert1 KEYSW, K1 KEYSW, K10 KEYSW, K11 KEYSW, K12 KEYSW, K13 KEYSW, K14 KEYSW, K15 KEYSW, K16 KEYSW, K17 KEYSW, K18 KEYSW, K19 KEYSW, K2 KEYSW, K20 KEYSW, K21 KEYSW, K22 KEYSW, K22-spacer1 KEYSW, K22-stepped1 KEYSW, K23 KEYSW, K24 KEYSW, K25 KEYSW, K26 KEYSW, K27 KEYSW, K28 KEYSW, K29 KEYSW, K3 KEYSW, K3-2uVert1 KEYSW, K30 KEYSW, K31 KEYSW, K32 KEYSW, K33 KEYSW, K34 KEYSW, K35 KEYSW, K35-2uVert1 KEYSW, K36 KEYSW, K37 KEYSW, K38 KEYSW, K38-2uVert1 KEYSW, K39 KEYSW, K39-spacer1 KEYSW, K4 KEYSW, K4-spacer1 KEYSW, K40 KEYSW, K41 KEYSW, K42 KEYSW, K43 KEYSW, K44 KEYSW, K45 KEYSW, K46 KEYSW, K47 KEYSW, K48 KEYSW, K49 KEYSW, K5 KEYSW, K50 KEYSW, K51 KEYSW, K52 KEYSW, K52-1u1 KEYSW, K53 KEYSW, K54 KEYSW, K54-2u1 KEYSW, K55 KEYSW, K55-1.25 KEYSW, K55-spacer1 KEYSW, K55-spacer2 KEYSW, K56 KEYSW, K56-1.25 KEYSW, K57 KEYSW, K57-1.25 KEYSW, K57-1.5u1 KEYSW, K57-1u1 KEYSW, K58 KEYSW, K58-6u1 KEYSW, K58for1.25Row1 KEYSW, K59 KEYSW, K59-1.25u1 KEYSW, K59-7u1 KEYSW, K59Alt1 KEYSW, K6 KEYSW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

Commit message: some more tweaks on keyboards
Parts:
- K0-2uVert1, K35-2uVert1: footprint MX_Only:MXOnly-2U-NoLED -> MX_Only:MXOnly-2U-ReversedStabilizers-NoLED
Changed lines of the file:
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@@
       (effects (font (size 1.524 1.524)) hide)
     )
-    (property "Footprint" "MX_Only:MXOnly-2U-NoLED" (id 2) (at 25.4 29.21 0)
+    (property "Footprint" "MX_Only:MXOnly-2U-ReversedStabilizers-NoLED" (id 2) (at 25.4 29.21 0)
       (effects (font (size 1.524 1.524)) hide)
     )
@@
       (effects (font (size 1.524 1.524)) hide)
     )
-    (property "Footprint" "MX_Only:MXOnly-2U-NoLED" (id 2) (at 38.1 91.44 0)
+    (property "Footprint" "MX_Only:MXOnly-2U-ReversedStabilizers-NoLED" (id 2) (at 38.1 91.44 0)
       (effects (font (size 1.524 1.524)) hide)
     )
@@
     )
     (path "/b6892239-8cc4-4239-9f6b-bd2be89fdd6c"
-      (reference "K0-2uVert1") (unit 1) (value "KEYSW") (footprint "MX_Only:MXOnly-2U-NoLED")
+      (reference "K0-2uVert1") (unit 1) (value "KEYSW") (footprint "MX_Only:MXOnly-2U-ReversedStabilizers-NoLED")
     )
     (path "/00000000-0000-0000-0000-000062166a86"
@@
     )
     (path "/d631fecf-1e8a-41e4-b2c3-fff52c91425c"
-      (reference "K35-2uVert1") (unit 1) (value "KEYSW") (footprint "MX_Only:MXOnly-2U-NoLED")
+      (reference "K35-2uVert1") (unit 1) (value "KEYSW") (footprint "MX_Only:MXOnly-2U-ReversedStabilizers-NoLED")
     )
     (path "/00000000-0000-0000-0000-000062166a6c"
