File: Longboi/longboi-plate.kicad_pcb (KiCad board)
At the start: 2 copper layers, 383 x 78.2 mm, 0 parts

Commit message: fix bug in longboi...
key38 was not schematiced right
Other:
- board size 383 x 78.2 mm -> 384 x 79.2 mm

Commit message: now purchasing
Parts:
- added G1: dotlen, Images:dotlen_14, F.Cu at (391.6, 75.7)
- added G2: string_dotlen, Images:string-dotlen_90mm_high, B.Cu at (204.4, 69.5)
Other:
- board size 384 x 79.2 mm -> 381 x 76.2 mm
- board text added: "'"
- board text added: ","
- board text added: "."
- board text added: ";"
- board text added: "?"
- board text added: "A"
- board text added: "B"
- board text added: "C"
- board text added: "D"
- board text added: "E"
- board text added: "F"
- board text added: "G"
- board text added: "H"
- board text added: "I"
- board text added: "J"
- board text added: "K"
- board text added: "L"
- board text added: "M"
- board text added: "N"
- board text added: "O"
- board text added: "P"
- board text added: "Q"
- board text added: "R"
- board text added: "S"
- board text added: "T"
- board text added: "U"
- board text added: "V"
- board text added: "W"
- board text added: "X"
- board text added: "Y"
- board text added: "Z"
- board text added: "["
- board text added: "]"
