File: Array/throughhole.kicad_pcb (KiCad board)
At the start: 2 copper layers, 383 x 102 mm, 185 parts, among them J2 ICSP_Header, K0 KEYSW, K1 KEYSW, K10 KEYSW, K11 KEYSW, K12 KEYSW, K13 KEYSW, K14 KEYSW, K15 KEYSW, K16 KEYSW, K17 KEYSW, K18 KEYSW, K19 KEYSW, K2 KEYSW, K20 KEYSW, K21 KEYSW, K22 KEYSW, K22-stepped1 KEYSW, K23 KEYSW, K24 KEYSW, K25 KEYSW, K26 KEYSW, K27 KEYSW, K28 KEYSW, K29 KEYSW, K3 KEYSW, K3-2uVert1 KEYSW, K30 KEYSW, K31 KEYSW, K32 KEYSW, K33 KEYSW, K34 KEYSW, K35 KEYSW, K36 KEYSW, K37 KEYSW, K38 KEYSW, K38-2uVert1 KEYSW, K39 KEYSW, K4 KEYSW, K40 KEYSW, K41 KEYSW, K42 KEYSW, K43 KEYSW, K44 KEYSW, K45 KEYSW, K46 KEYSW, K47 KEYSW, K48 KEYSW, K49 KEYSW, K5 KEYSW, K50 KEYSW, K51 KEYSW, K52 KEYSW, K53 KEYSW, K54 KEYSW, K55 KEYSW, K55-1.25 KEYSW, K56 KEYSW, K56-1.25 KEYSW, K57 KEYSW, K57-1.25 KEYSW, K57-1.5u1 KEYSW, K58 KEYSW, K58-6u1 KEYSW, K58for1.25Row1 KEYSW, K59 KEYSW, K59-1.25u1 KEYSW, K59-7u1 KEYSW, K59Alt1 KEYSW, K6 KEYSW, K60 KEYSW, K60Alt1 KEYSW, K61 KEYSW, K61-1.5u1 KEYSW, K62 KEYSW, K62-1.5u1 KEYSW, K63 KEYSW, K64 KEYSW, K65 KEYSW, K66 KEYSW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

Commit message: some array changes
Parts:
- removed G***: LOGO, Images:array_dotlen_logo_526
- added Array_Logo2: Array_Logo, Images:array_dotlen_logo_526, B.Cu at (184.6, 110.5)
- U1: renamed from ATmega32U4; value ATmega32U4-AU -> ATmega32U4-MUR
- moved K68 1.27 mm to (381.0, 104.8)
Routing:
- net /Col_17: track 225.9 -> 210.2 mm
- net /Col_9: track 140.0 -> 151.1 mm
- net /Col_15: track 268.7 -> 276.5 mm
- net Net-(D21-Pad2): track 80.0 -> 84.5 mm
- net /Col_16: track 261.5 -> 265.2 mm
- net /Col_10: track 170.5 -> 166.9 mm
- net /Col_12: track 145.2 -> 142.4 mm
- net /Col_3: track 444.5 -> 447.0 mm
- net Net-(D63-Pad2): track 188.7 -> 190.8 mm
- net /Col_13: track 111.0 -> 109.6 mm
- net /Col_8: track 207.1 -> 205.9 mm
- net /Col_7: track 198.9 -> 197.6 mm
- net Net-(D46-Pad2): track 127.8 -> 127.3 mm
