File: List/list.kicad_pcb (KiCad board)
At the start: 2 copper layers, 373.5 x 102 mm, 227 parts, among them J2 ICSP_Header, K0 KEYSW, K0-2uVert1 KEYSW, K1 KEYSW, K10 KEYSW, K11 KEYSW, K12 KEYSW, K13 KEYSW, K14 KEYSW, K15 KEYSW, K16 KEYSW, K17 KEYSW, K18 KEYSW, K19 KEYSW, K2 KEYSW, K20 KEYSW, K21 KEYSW, K22 KEYSW, K22-stepped1 KEYSW, K23 KEYSW, K24 KEYSW, K25 KEYSW, K26 KEYSW, K27 KEYSW, K28 KEYSW, K29 KEYSW, K3 KEYSW, K3-2uVert1 KEYSW, K30 KEYSW, K31 KEYSW, K32 KEYSW, K33 KEYSW, K34 KEYSW, K35 KEYSW, K36 KEYSW, K37 KEYSW, K38 KEYSW, K38-2uVert1 KEYSW, K39 KEYSW, K4 KEYSW, K40 KEYSW, K41 KEYSW, K42 KEYSW, K43 KEYSW, K44 KEYSW, K45 KEYSW, K46 KEYSW, K47 KEYSW, K48 KEYSW, K49 KEYSW, K5 KEYSW, K50 KEYSW, K51 KEYSW, K53 KEYSW, K53-2 KEYSW, K54 KEYSW, K54-2u1 KEYSW, K55 KEYSW, K55-1.25 KEYSW, K56 KEYSW, K56-1.25 KEYSW, K57 KEYSW, K57-1.25 KEYSW, K57-1.5u1 KEYSW, K57-1u1 KEYSW, K58 KEYSW, K58-6u1 KEYSW, K58for1.25Row1 KEYSW, K59 KEYSW, K59-1.25u1 KEYSW, K59-7u1 KEYSW, K59Alt1 KEYSW, K6 KEYSW, K60 KEYSW, K60Alt1 KEYSW, K61 KEYSW, K61-1.25u1 KEYSW, K61-1.5u1 KEYSW, K62 KEYSW, K62-1.25u1 KEYSW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

Commit message: probably buying all three now
Parts:
- removed D52, D66, D67, D68, D88: SOD-323F, Diode_SMD:D_SOD-323F
- removed H6, H7, H8, H9: MountingHole, random-keyboard-parts:M2 Mounting Hole
- removed K0-2uVert1: KEYSW, MX_Only:MXOnly-2U-NoLED
- added K17_Iso_1u1: KEYSW, MX_Only:MXOnly-1U-NoLED, F.Cu at (268.2, 48.9)
- added K34_iso1: KEYSW, MX_Only:MXOnly-ISO-ROTATED-ReversedStabilizers-NoLED, F.Cu at (289.6, 39.4)
- added SW2: Rotary_Encoder_Switch, random-keyboard-parts:RotaryEncoder_Alps_EC11E-Switch_Vertical_H20mm_MX-1U, F.Cu at (377.7, 10.8)
- G2: renamed from Ge; footprint Images:map-dotlen108mm -> Images:list-dotlen_90mm_high
- G3: footprint Images:Map_5.7mm_high -> Images:List_5mm_high
- K34, K39: footprint MX_Only:MXOnly-2.25U-ReversedStabilizers-NoLED -> MX_Only:MXOnly-2.25U-NoLED
- moved D35 295.3 mm to (316.8, 71.7)
- moved D70 295.3 mm to (316.7, 14.5)
- moved D0 295.3 mm to (316.7, 33.6)
- moved D18 295.3 mm to (316.7, 52.6)
- moved G2 30.9 mm to (189.9, 56.0)
- moved H5 9.53 mm to (182.4, 58.4)
- moved D51 6.74 mm to (292.9, 76.4)
- moved D64 6.74 mm to (273.9, 95.4)
- moved R6 5.11 mm to (273.5, 7.52), turned to 90 degrees
- moved P1 1.43 mm to (263.4, 4.32)
- moved G3 1.40 mm to (94.5, 85.6)
- moved R2 1.23 mm to (262.2, 14.1)
- moved R3 1.23 mm to (264.2, 14.1)
- moved R5 1.23 mm to (252.4, 4.93)
- moved F1 1.23 mm to (261.1, 19.4)
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Routing:
- net Net-(D19-Pad2): track 743.2 -> 5.33 mm, vias 3 -> 0
- net /Col_1: track 542.0 -> 216.2 mm, vias 2 -> 0
- net GND: track 5.15 -> 312.9 mm, vias 0 -> 4
- net Net-(D71-Pad2): track 269.9 -> 5.15 mm, vias 6 -> 0
- net /Col_8: track 0.00 -> 263.1 mm, vias 0 -> 1
- net /Col_2: track 503.9 -> 244.1 mm, vias 2 -> 0
- net /Col_9: track 0.00 -> 258.1 mm, vias 0 -> 1
- net /Col_10: track 0.00 -> 244.5 mm, vias 0 -> 1
- net /Col_0: track 414.6 -> 182.0 mm, vias 1 -> 0
- net Rotary_A: track 0.00 -> 196.8 mm, vias 0 -> 1
- net /Col_3: track 443.7 -> 271.7 mm, vias 1 -> 0
- net /Col_14: track 0.00 -> 152.6 mm, vias 0 -> 1
- net Net-(D37-Pad2): track 90.9 -> 5.33 mm, vias 2 -> 0
- net /Row_2: track 439.4 -> 364.9 mm, vias 2 -> 4
- net /Row_3: track 455.6 -> 388.3 mm, vias 0 -> 2
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Other:
- board size 373.5 x 102 mm -> 371.5 x 100 mm
- board text added: "1U (ISO)"
- board text added: "ISO"
