File: List/list.kicad_sch (KiCad schematic)
At the start: 234 parts, among them J2 ICSP_Header, K0 KEYSW, K0-2uVert1 KEYSW, K1 KEYSW, K10 KEYSW, K11 KEYSW, K12 KEYSW, K13 KEYSW, K14 KEYSW, K15 KEYSW, K16 KEYSW, K17 KEYSW, K18 KEYSW, K19 KEYSW, K2 KEYSW, K20 KEYSW, K21 KEYSW, K22 KEYSW, K22-stepped1 KEYSW, K23 KEYSW, K24 KEYSW, K25 KEYSW, K26 KEYSW, K27 KEYSW, K28 KEYSW, K29 KEYSW, K3 KEYSW, K3-2uVert1 KEYSW, K30 KEYSW, K31 KEYSW, K32 KEYSW, K33 KEYSW, K34 KEYSW, K35 KEYSW, K35-2uVert1 KEYSW, K36 KEYSW, K37 KEYSW, K38 KEYSW, K38-2uVert1 KEYSW, K39 KEYSW, K4 KEYSW, K40 KEYSW, K41 KEYSW, K42 KEYSW, K43 KEYSW, K44 KEYSW, K45 KEYSW, K46 KEYSW, K47 KEYSW, K48 KEYSW, K49 KEYSW, K5 KEYSW, K50 KEYSW, K51 KEYSW, K52 KEYSW, K52-1u1 KEYSW, K53 KEYSW, K53-2 KEYSW, K54 KEYSW, K54-2u1 KEYSW, K55 KEYSW, K55-1.25 KEYSW, K56 KEYSW, K56-1.25 KEYSW, K57 KEYSW, K57-1.25 KEYSW, K57-1.5u1 KEYSW, K57-1u1 KEYSW, K58 KEYSW, K58-6u1 KEYSW, K58for1.25Row1 KEYSW, K59 KEYSW, K59-1.25u1 KEYSW, K59-7u1 KEYSW, K59Alt1 KEYSW, K6 KEYSW, K60 KEYSW, K60Alt1 KEYSW, K61 KEYSW, K61-1.25u1 KEYSW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

Commit message: probably buying all three now
Parts:
- removed D52, D66, D67, D68, D88: SOD-323F, Diode_SMD:D_SOD-323F, symbol Device:D
- removed H6, H7, H8, H9: MountingHole, random-keyboard-parts:M2 Mounting Hole, symbol Mechanical:MountingHole
- removed K0-2uVert1, K35-2uVert1: KEYSW, MX_Only:MXOnly-2U-NoLED, symbol Switch:SW_Push
- removed K52: KEYSW, MX_Only:MXOnly-2U-ReversedStabilizers-NoLED, symbol Switch:SW_Push
- removed K52-1u1, K66, K67, K68, K88: KEYSW, MX_Only:MXOnly-1U-NoLED, symbol Switch:SW_Push
- removed SW3: Rotary_Encoder_Switch, random-keyboard-parts:RotaryEncoder_Alps_EC11E-Switch_Vertical_H20mm_MX-1U, symbol Device:Rotary_Encoder_Switch
- added K17_Iso_1u1: KEYSW, MX_Only:MXOnly-1U-NoLED, symbol Switch:SW_Push
- added K34_iso1: KEYSW, MX_Only:MXOnly-ISO-ROTATED-ReversedStabilizers-NoLED, symbol Switch:SW_Push
- added SW2: Rotary_Encoder_Switch, random-keyboard-parts:RotaryEncoder_Alps_EC11E-Switch_Vertical_H20mm_MX-1U, symbol Device:Rotary_Encoder_Switch
- G2: footprint Images:map-dotlen108mm -> Images:list-dotlen_90mm_high
- G3: footprint Images:Map_5.7mm_high -> Images:List_5mm_high
- K34, K39: footprint MX_Only:MXOnly-2.25U-ReversedStabilizers-NoLED -> MX_Only:MXOnly-2.25U-NoLED
Connections:
- net Col_16: now also K34_iso1.2
- net Col_17: now also K17_Iso_1u1.2
- net Col_3: now also SW2.S1
- net GND: now also SW2.C
- net Rotary_A: now also SW2.A
- net Rotary_B: now also SW2.B
- net at D34.2 (A), K34.1: now also K34_iso1.1
- net at D17.2 (A), K17.1: now also K17_Iso_1u1.1
- net at D73.2 (A), K73.1: now also SW2.S2
Other:
- moved on the sheet: D0, D1, D10, D11, D12, D13, D14, D15, D16, D17, D18, D19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
