File: List/list-plate.kicad_pcb (KiCad board)
At the start: 2 copper layers, 371.5 x 100 mm, 7 parts

Commit message: Update List and Map
Update List and Map
Other:
- board size 371.5 x 100 mm -> 371.5 x 104.8 mm
