File: Map/map.kicad_pcb (KiCad board)
At the start: 2 copper layers, 392.5 x 97.3 mm, 234 parts, among them J2 ICSP_Header, K0 KEYSW, K0-2uVert1 KEYSW, K1 KEYSW, K10 KEYSW, K11 KEYSW, K12 KEYSW, K13 KEYSW, K14 KEYSW, K15 KEYSW, K16 KEYSW, K17 KEYSW, K18 KEYSW, K19 KEYSW, K2 KEYSW, K20 KEYSW, K21 KEYSW, K22 KEYSW, K22-stepped1 KEYSW, K23 KEYSW, K24 KEYSW, K25 KEYSW, K26 KEYSW, K27 KEYSW, K28 KEYSW, K29 KEYSW, K3 KEYSW, K3-2uVert1 KEYSW, K30 KEYSW, K31 KEYSW, K32 KEYSW, K33 KEYSW, K34 KEYSW, K35 KEYSW, K35-2uVert1 KEYSW, K36 KEYSW, K37 KEYSW, K38 KEYSW, K38-2uVert1 KEYSW, K39 KEYSW, K4 KEYSW, K40 KEYSW, K41 KEYSW, K42 KEYSW, K43 KEYSW, K44 KEYSW, K45 KEYSW, K46 KEYSW, K47 KEYSW, K48 KEYSW, K49 KEYSW, K5 KEYSW, K50 KEYSW, K51 KEYSW, K52 KEYSW, K52-1u1 KEYSW, K53 KEYSW, K53-2 KEYSW, K54 KEYSW, K54-2u1 KEYSW, K55 KEYSW, K55-1.25 KEYSW, K56 KEYSW, K56-1.25 KEYSW, K57 KEYSW, K57-1.25 KEYSW, K57-1.5u1 KEYSW, K57-1u1 KEYSW, K58 KEYSW, K58-6u1 KEYSW, K58for1.25Row1 KEYSW, K59 KEYSW, K59-1.25u1 KEYSW, K59-7u1 KEYSW, K59Alt1 KEYSW, K6 KEYSW, K60 KEYSW, K60Alt1 KEYSW, K61 KEYSW, K61-1.25u1 KEYSW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

Commit message: CLean up gitignore, update map
Parts:
- added G***: LOGO, Images:beebo_12mm, F.Cu at (319.5, 57.4)
Routing:
- net /Row_3: track 470.8 -> 455.6 mm
- net /Col_4: track 307.2 -> 303.0 mm
- net /Col_17: track 198.9 -> 195.9 mm

Commit message: update map, delete some old fi les
Parts:
- moved G*** 211.6 mm to (108.1, 67.5)
Routing:
- net Rotary_A: track 161.4 -> 157.9 mm
- net Rotary_B: track 149.4 -> 148.3 mm

Commit message: clean up map and string with prototype fixes
Parts:
- removed K57-1u1: KEYSW, MX_Only:MXOnly-1U-NoLED
- added REF**: MountingHole_4mm, MountingHole:MountingHole_4mm, F.Cu at (94.3, 20.3)
- added REF**: MountingHole_4mm, MountingHole:MountingHole_4mm, F.Cu at (94.3, 77.5)
- K34: footprint MX_Only:MXOnly-2.25U-ReversedStabilizers-NoLED -> MX_Only:MXOnly-2.25U-NoLED
- moved H3 30.5 mm to (115.8, 20.3)
- moved H2 23.8 mm to (115.8, 77.5)
- moved H1 19.6 mm to (325.3, 20.3)
- moved C8 4.76 mm to (342.2, 57.4)
- moved D16 4.76 mm to (340.6, 33.6)
- moved D17 4.76 mm to (364.4, 33.7)
- moved D30 4.76 mm to (269.1, 52.6)
- moved D49 4.76 mm to (316.7, 71.6)
- moved D62 4.76 mm to (312.0, 90.7)
- moved D66 4.76 mm to (388.2, 33.7)
- moved D67 4.76 mm to (388.2, 52.7)
- moved D68 4.76 mm to (388.2, 71.6)
- moved D69 4.76 mm to (388.2, 90.7)
- moved D84 4.76 mm to (292.9, 14.5)
- moved D88 4.76 mm to (388.2, 14.5)
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- renumbered Ge to G2
Routing:
- net /Col_1: track 370.6 -> 365.8 mm
- net /Col_3: track 348.5 -> 343.7 mm
- net /Row_2: track 439.4 -> 434.6 mm
- net /Col_2: track 355.7 -> 351.0 mm
- net /Col_0: track 414.6 -> 409.8 mm
- net /Col_14: track 148.2 -> 151.9 mm
- net /Row_1: track 450.7 -> 447.8 mm
- net /Row_4: track 401.1 -> 403.8 mm
- net /Col_17: track 195.7 -> 197.8 mm
- net /Col_4: track 303.0 -> 304.6 mm
- net /Col_15: track 144.6 -> 145.2 mm
Other:
- board size 392.5 x 97.3 mm -> 387.8 x 97.3 mm

Commit message: moreupdates to tweak the two keyboards
Parts:
- removed REF** (x2): MountingHole_4mm, MountingHole:MountingHole_4mm
- added K17_Iso_1u1: KEYSW, MX_Only:MXOnly-1U-NoLED, F.Cu at (349.1, 48.9)
- added K34_iso1: KEYSW, MX_Only:MXOnly-ISO-ROTATED-ReversedStabilizers-NoLED, F.Cu at (370.6, 39.4)
- K0-2uVert1, K35-2uVert1: footprint MX_Only:MXOnly-2U-NoLED -> MX_Only:MXOnly-2U-ReversedStabilizers-NoLED
- turned K0-2uVert1 to -90 degrees
- turned K35-2uVert1 to -90 degrees
Routing:
- net /Col_17: track 197.8 -> 228.0 mm
- net Net-(D17-Pad2): track 5.33 -> 32.3 mm
- net Net-(D34-Pad2): track 5.15 -> 25.5 mm
- net /Col_16: track 142.2 -> 156.0 mm
- net /Col_0: track 409.8 -> 397.3 mm
- net Net-(D35-Pad2): track 19.8 -> 13.2 mm
- net GND: track 249.8 -> 254.4 mm
- net VCC: track 133.4 -> 131.1 mm
- net /Row_2: track 434.6 -> 435.9 mm
- net /Row_0: track 410.2 -> 411.4 mm
Other:
- board text added: "1U (ISO)"
- board text added: "ISO"

Commit message: some more tweaks on keyboards
Parts:
- moved G*** 0.37 mm to (103.6, 67.2)

Commit message: probably buying all three now
Parts:
- removed H6, H7, H8, H9: MountingHole, random-keyboard-parts:M2 Mounting Hole
- moved R6 1.62 mm to (355.8, 4.27)
- moved P1 1.42 mm to (344.2, 4.32)
- moved F1 1.26 mm to (342.1, 19.4)
- moved R2 1.26 mm to (343.2, 14.2)
- moved R3 1.26 mm to (345.2, 14.1)
Routing:
- net GND: track 254.4 -> 243.6 mm
- net Net-(P1-PadB5): track 13.5 -> 11.9 mm
- net Net-(R2-Pad1): track 54.6 -> 53.4 mm
- net Net-(R3-Pad1): track 54.8 -> 53.5 mm
- net Net-(P1-PadA5): track 11.1 -> 11.7 mm
Other:
- board size 387.8 x 97.3 mm -> 385.8 x 95.3 mm
