File: Map/map.kicad_sch (KiCad schematic)
At the start: 234 parts, among them J2 ICSP_Header, K0 KEYSW, K0-2uVert1 KEYSW, K1 KEYSW, K10 KEYSW, K11 KEYSW, K12 KEYSW, K13 KEYSW, K14 KEYSW, K15 KEYSW, K16 KEYSW, K17 KEYSW, K18 KEYSW, K19 KEYSW, K2 KEYSW, K20 KEYSW, K21 KEYSW, K22 KEYSW, K22-stepped1 KEYSW, K23 KEYSW, K24 KEYSW, K25 KEYSW, K26 KEYSW, K27 KEYSW, K28 KEYSW, K29 KEYSW, K3 KEYSW, K3-2uVert1 KEYSW, K30 KEYSW, K31 KEYSW, K32 KEYSW, K33 KEYSW, K34 KEYSW, K35 KEYSW, K35-2uVert1 KEYSW, K36 KEYSW, K37 KEYSW, K38 KEYSW, K38-2uVert1 KEYSW, K39 KEYSW, K4 KEYSW, K40 KEYSW, K41 KEYSW, K42 KEYSW, K43 KEYSW, K44 KEYSW, K45 KEYSW, K46 KEYSW, K47 KEYSW, K48 KEYSW, K49 KEYSW, K5 KEYSW, K50 KEYSW, K51 KEYSW, K52 KEYSW, K52-1u1 KEYSW, K53 KEYSW, K53-2 KEYSW, K54 KEYSW, K54-2u1 KEYSW, K55 KEYSW, K55-1.25 KEYSW, K56 KEYSW, K56-1.25 KEYSW, K57 KEYSW, K57-1.25 KEYSW, K57-1.5u1 KEYSW, K57-1u1 KEYSW, K58 KEYSW, K58-6u1 KEYSW, K58for1.25Row1 KEYSW, K59 KEYSW, K59-1.25u1 KEYSW, K59-7u1 KEYSW, K59Alt1 KEYSW, K6 KEYSW, K60 KEYSW, K60Alt1 KEYSW, K61 KEYSW, K61-1.25u1 KEYSW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

Commit message: CLean up gitignore, update map
Parts:
- G1: symbol Graphic:dotlen -> Dotlen_Logos:dotlen
- G2: footprint Images:string-dotlen_90mm_high -> Images:map-dotlen108mm; symbol string:string_dotlen -> Dotlen_Logos:map-dotlen_12mm
- G3: footprint Images:String_5.7mm_high -> Images:Map_5.7mm_high; symbol string:string -> Dotlen_Logos:map_5.7mm
Changed lines of the file:
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@@
     (stroke (width 0) (type default) (color 0 0 0 0))
   )
-  (wire (pts (xy 87.63 25.4) (xy 90.17 25.4))
-    (stroke (width 0) (type default) (color 0 0 0 0))
-  )
   (wire (pts (xy 152.4 229.87) (xy 152.4 218.44))
     (stroke (width 0) (type default) (color 0 0 0 0))
@@
     (pin "2")
   )
-  (symbol (lib_id "string:string") (at 250.19 243.84 0) (unit 1)
+  (symbol (lib_id "Dotlen_Logos:map_5.7mm") (at 250.19 241.3 0) (unit 1)
     (in_bom yes) (on_board yes)
-    (property "Reference" "G3" (id 0) (at 258.953 242.697 0)
+    (property "Reference" "G3" (id 0) (at 258.953 240.157 0)
       (effects (font (size 1.524 1.524)) (justify left))
     )
-    (property "Value" "string" (id 1) (at 250.19 241.7572 0)
+    (property "Value" "string" (id 1) (at 250.19 239.2172 0)
       (effects (font (size 1.524 1.524)) hide)
     )
-    (property "Footprint" "Images:String_5.7mm_high" (id 2) (at 258.953 245.1862 0)
-      (effects (font (size 1.27 1.27)) (justify left))
-    )
-    (property "Datasheet" "" (id 3) (at 250.19 243.84 0)
+    (property "Footprint" "Images:Map_5.7mm_high" (id 2) (at 250.19 243.84 0))
+    (property "Datasheet" "" (id 3) (at 250.19 241.3 0)
       (effects (font (size 1.27 1.27)) hide)
     )
   )
-  (symbol (lib_id "string:string_dotlen") (at 265.43 259.08 0) (unit 1)
+  (symbol (lib_id "Dotlen_Logos:map-dotlen_12mm") (at 265.43 259.08 0) (unit 1)
     (in_bom yes) (on_board yes)
     (property "Reference" "G2" (id 0) (at 265.43 251.9172 0)
@@
       (effects (font (size 1.524 1.524)) hide)
     )
-    (property "Footprint" "Images:string-dotlen_90mm_high" (id 2) (at 265.43 254.4064 0))
+    (property "Footprint" "Images:map-dotlen108mm" (id 2) (at 265.43 259.08 0)
+      (effects (font (size 1.27 1.27)) hide)
+    )
     (property "Datasheet" "" (id 3) (at 265.43 259.08 0)
       (effects (font (size 1.27 1.27)) hide)
@@
     (pin "2")
   )
-  (symbol (lib_id "Graphic:dotlen") (at 274.32 243.84 0) (unit 1)
+  (symbol (lib_id "Dotlen_Logos:dotlen") (at 274.32 243.84 0) (unit 1)
     (in_bom yes) (on_board yes)
     (property "Reference" "G1" (id 0) (at 274.2946 237.0582 0)
@@
       (effects (font (size 1.524 1.524)) hide)
     )
-    (property "Footprint" "Images:dotlen_14" (id 2) (at 274.2946 239.5474 0))
+    (property "Footprint" "Images:dotlen_14" (id 2) (at 274.32 247.65 0))
     (property "Datasheet" "" (id 3) (at 274.32 243.84 0)
       (effects (font (size 1.27 1.27)) hide)
@@
     )
     (path "/00000000-0000-0000-0000-000061d579ec"
-      (reference "G2") (unit 1) (value "string_dotlen") (footprint "Images:string-dotlen_90mm_high")
+      (reference "G2") (unit 1) (value "string_dotlen") (footprint "Images:map-dotlen108mm")
     )
     (path "/00000000-0000-0000-0000-000061d557a5"
-      (reference "G3") (unit 1) (value "string") (footprint "Images:String_5.7mm_high")
+      (reference "G3") (unit 1) (value "string") (footprint "Images:Map_5.7mm_high")
     )
     (path "/00000000-0000-0000-0000-000062166a34"

Commit message: clean up map and string with prototype fixes
Parts:
- removed K57-1u1: KEYSW, MX_Only:MXOnly-1U-NoLED, symbol Switch:SW_Push
- K34: footprint MX_Only:MXOnly-2.25U-ReversedStabilizers-NoLED -> MX_Only:MXOnly-2.25U-NoLED
Other:
- moved on the sheet: D0, D1, D18, D19, D2, D20, D21, D22, D3, D35, D36, D37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

Commit message: moreupdates to tweak the two keyboards
Parts:
- added K17_Iso_1u1: KEYSW, MX_Only:MXOnly-1U-NoLED, symbol Switch:SW_Push
- added K34_iso1: KEYSW, MX_Only:MXOnly-ISO-ROTATED-ReversedStabilizers-NoLED, symbol Switch:SW_Push
- K0-2uVert1, K35-2uVert1: footprint MX_Only:MXOnly-2U-NoLED -> MX_Only:MXOnly-2U-ReversedStabilizers-NoLED
Connections:
- net Col_16: now also K34_iso1.2
- net Col_17: now also K17_Iso_1u1.2
- net at D34.2 (A), K34.1: now also K34_iso1.1
- net at D17.2 (A), K17.1: now also K17_Iso_1u1.1
Changed lines of the file:
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@@
   (junction (at 161.29 157.48) (diameter 0) (color 0 0 0 0)
   )
+  (junction (at 369.57 52.07) (diameter 0) (color 0 0 0 0)
+  )
   (junction (at 281.94 157.48) (diameter 0) (color 0 0 0 0)
   )
@@
   (junction (at 105.41 251.46) (diameter 0) (color 0 0 0 0)
   )
+  (junction (at 360.68 76.2) (diameter 0) (color 0 0 0 0)
+  )
   (junction (at 311.15 105.41) (diameter 0) (color 0 0 0 0)
   )
@@
     (stroke (width 0) (type default) (color 0 0 0 0))
   )
+  (wire (pts (xy 370.84 72.39) (xy 370.84 76.2))
+    (stroke (width 0) (type default) (color 0 0 0 0))
+  )
   (wire (pts (xy 209.55 33.02) (xy 229.87 33.02))
     (stroke (width 0) (type default) (color 0 0 0 0))
@@
     (stroke (width 0) (type default) (color 0 0 0 0))
   )
+  (wire (pts (xy 360.68 72.39) (xy 360.68 76.2))
+    (stroke (width 0) (type default) (color 0 0 0 0))
+  )
   (wire (pts (xy 134.62 242.57) (xy 130.81 242.57))
     (stroke (width 0) (type default) (color 0 0 0 0))
@@
     (stroke (width 0) (type default) (color 0 0 0 0))
   )
+  (wire (pts (xy 379.73 48.26) (xy 379.73 52.07))
+    (stroke (width 0) (type default) (color 0 0 0 0))
+  )
   (wire (pts (xy 185.42 128.27) (xy 185.42 134.62))
     (stroke (width 0) (type default) (color 0 0 0 0))
@@
     (stroke (width 0) (type default) (color 0 0 0 0))
   )
+  (wire (pts (xy 369.57 48.26) (xy 369.57 52.07))
+    (stroke (width 0) (type default) (color 0 0 0 0))
+  )
   (wire (pts (xy 168.91 33.02) (xy 189.23 33.02))
     (stroke (width 0) (type default) (color 0 0 0 0))
@@
     (pin "2")
   )
+  (symbol (lib_id "Switch:SW_Push") (at 365.76 72.39 0) (unit 1)
+    (in_bom yes) (on_board yes)
+    (property "Reference" "K34_iso1" (id 0) (at 365.76 66.4718 0)
+      (effects (font (size 1.524 1.524)))
+    )
+    (property "Value" "KEYSW" (id 1) (at 365.76 74.93 0)
+      (effects (font (size 1.524 1.524)) hide)
+    )
+    (property "Footprint" "MX_Only:MXOnly-ISO-ROTATED-ReversedStabilizers-NoLED" (id 2) (at 365.76 72.39 0)
+      (effects (font (size 1.524 1.524)) hide)
+    )
+    (property "Datasheet" "" (id 3) (at 365.76 72.39 0)
+      (effects (font (size 1.524 1.524)))
+    )
+    (pin "1")
+    (pin "2")
+  )
   (symbol (lib_id "Device:D") (at 209.55 29.21 90) (unit 1)
     (in_bom yes) (on_board yes)
@@
       (effects (font (size 1.524 1.524)) hide)
     )
-    (property "Footprint" "MX_Only:MXOnly-2U-NoLED" (id 2) (at 25.4 52.07 0)
+    (property "Footprint" "MX_Only:MXOnly-2U-ReversedStabilizers-NoLED" (id 2) (at 25.4 52.07 0)
       (effects (font (size 1.524 1.524)) hide)
     )
@@
       (effects (font (size 1.524 1.524)) hide)
     )
-    (property "Footprint" "MX_Only:MXOnly-2U-NoLED" (id 2) (at 24.13 96.52 0)
+    (property "Footprint" "MX_Only:MXOnly-2U-ReversedStabilizers-NoLED" (id 2) (at 24.13 96.52 0)
       (effects (font (size 1.524 1.524)) hide)
     )
@@
     (pin "2")
   )
+  (symbol (lib_id "Switch:SW_Push") (at 374.65 48.26 0) (unit 1)
+    (in_bom yes) (on_board yes)
+    (property "Reference" "K17_Iso_1u1" (id 0) (at 374.65 42.3418 0)
+      (effects (font (size 1.524 1.524)))
+    )
+    (property "Value" "KEYSW" (id 1) (at 374.65 50.8 0)
+      (effects (font (size 1.524 1.524)) hide)
+    )
+    (property "Footprint" "MX_Only:MXOnly-1U-NoLED" (id 2) (at 374.65 48.26 0)
+      (effects (font (size 1.524 1.524)) hide)
+    )
+    (property "Datasheet" "" (id 3) (at 374.65 48.26 0)
+      (effects (font (size 1.524 1.524)))
+    )
+    (pin "1")
+    (pin "2")
+  )
   (symbol (lib_id "Switch:SW_Push") (at 26.67 146.05 0) (unit 1)
     (in_bom yes) (on_board yes)
@@
     )
     (path "/359670f9-189a-4098-a82b-ec9037da56d1"
-      (reference "K0-2uVert1") (unit 1) (value "KEYSW") (footprint "MX_Only:MXOnly-2U-NoLED")
+      (reference "K0-2uVert1") (unit 1) (value "KEYSW") (footprint "MX_Only:MXOnly-2U-ReversedStabilizers-NoLED")
     )
     (path "/00000000-0000-0000-0000-000062166a86"
@@
       (reference "K17") (unit 1) (value "KEYSW") (footprint "MX_Only:MXOnly-1.5U-NoLED")
     )
+    (path "/9b03ade2-7747-4e96-bf1a-aba28ac085cc"
+      (reference "K17_Iso_1u1") (unit 1) (value "KEYSW") (footprint "MX_Only:MXOnly-1U-NoLED")
+    )
     (path "/00000000-0000-0000-0000-000061be6ab6"
       (reference "K18") (unit 1) (value "KEYSW") (footprint "MX_Only:MXOnly-1U-NoLED")
@@
       (reference "K34") (unit 1) (value "KEYSW") (footprint "MX_Only:MXOnly-2.25U-NoLED")
     )
+    (path "/20364b64-c482-49ea-bc80-e96543f69561"
+      (reference "K34_iso1") (unit 1) (value "KEYSW") (footprint "MX_Only:MXOnly-ISO-ROTATED-ReversedStabilizers-NoLED")
+    )
     (path "/00000000-0000-0000-0000-000062166a6d"
       (reference "K35") (unit 1) (value "KEYSW") (footprint "MX_Only:MXOnly-1U-NoLED")
     )
     (path "/5bc79adf-87d3-4257-937b-072dc80fee87"
-      (reference "K35-2uVert1") (unit 1) (value "KEYSW") (footprint "MX_Only:MXOnly-2U-NoLED")
+      (reference "K35-2uVert1") (unit 1) (value "KEYSW") (footprint "MX_Only:MXOnly-2U-ReversedStabilizers-NoLED")
     )
     (path "/00000000-0000-0000-0000-000062166a6c"

Commit message: probably buying all three now
Parts:
- removed H6, H7, H8, H9: MountingHole, random-keyboard-parts:M2 Mounting Hole, symbol Mechanical:MountingHole
Changed lines of the file:
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@@
   (junction (at 331.47 157.48) (diameter 0) (color 0 0 0 0)
   )
-  (junction (at 414.02 27.94) (diameter 0) (color 0 0 0 0)
-  )
   (junction (at 77.47 144.78) (diameter 0) (color 0 0 0 0)
   )
@@
     (pin "2")
   )
-  (symbol (lib_id "Mechanical:MountingHole") (at 39.37 189.23 0) (unit 1)
-    (in_bom yes) (on_board yes)
-    (property "Reference" "H7" (id 0) (at 41.91 188.0616 0)
-      (effects (font (size 1.27 1.27)) (justify left))
-    )
-    (property "Value" "MountingHole" (id 1) (at 41.91 190.373 0)
-      (effects (font (size 1.27 1.27)) (justify left))
-    )
-    (property "Footprint" "random-keyboard-parts:M2 Mounting Hole" (id 2) (at 39.37 189.23 0)
-      (effects (font (size 1.27 1.27)) hide)
-    )
-    (property "Datasheet" "~" (id 3) (at 39.37 189.23 0)
-      (effects (font (size 1.27 1.27)) hide)
-    )
-  )
   (symbol (lib_id "Device:D") (at 148.59 29.21 90) (unit 1)
     (in_bom yes) (on_board yes)
@@
     (pin "2")
   )
-  (symbol (lib_id "Mechanical:MountingHole") (at 60.96 177.8 0) (unit 1)
-    (in_bom yes) (on_board yes)
-    (property "Reference" "H8" (id 0) (at 63.5 176.6316 0)
-      (effects (font (size 1.27 1.27)) (justify left))
-    )
-    (property "Value" "MountingHole" (id 1) (at 63.5 178.943 0)
-      (effects (font (size 1.27 1.27)) (justify left))
-    )
-    (property "Footprint" "random-keyboard-parts:M2 Mounting Hole" (id 2) (at 60.96 177.8 0)
-      (effects (font (size 1.27 1.27)) hide)
-    )
-    (property "Datasheet" "~" (id 3) (at 60.96 177.8 0)
-      (effects (font (size 1.27 1.27)) hide)
-    )
-  )
-  (symbol (lib_id "Mechanical:MountingHole") (at 60.96 189.23 0) (unit 1)
-    (in_bom yes) (on_board yes)
-    (property "Reference" "H9" (id 0) (at 63.5 188.0616 0)
-      (effects (font (size 1.27 1.27)) (justify left))
-    )
-    (property "Value" "MountingHole" (id 1) (at 63.5 190.373 0)
-      (effects (font (size 1.27 1.27)) (justify left))
-    )
-    (property "Footprint" "random-keyboard-parts:M2 Mounting Hole" (id 2) (at 60.96 189.23 0)
-      (effects (font (size 1.27 1.27)) hide)
-    )
-    (property "Datasheet" "~" (id 3) (at 60.96 189.23 0)
-      (effects (font (size 1.27 1.27)) hide)
-    )
-  )
   (symbol (lib_id "Switch:SW_Push") (at 25.4 52.07 0) (unit 1)
     (in_bom yes) (on_board yes)
@@
     (pin "2")
   )
-  (symbol (lib_id "Mechanical:MountingHole") (at 39.37 177.8 0) (unit 1)
-    (in_bom yes) (on_board yes)
-    (property "Reference" "H6" (id 0) (at 41.91 176.6316 0)
-      (effects (font (size 1.27 1.27)) (justify left))
-    )
-    (property "Value" "MountingHole" (id 1) (at 41.91 178.943 0)
-      (effects (font (size 1.27 1.27)) (justify left))
-    )
-    (property "Footprint" "random-keyboard-parts:M2 Mounting Hole" (id 2) (at 39.37 177.8 0)
-      (effects (font (size 1.27 1.27)) hide)
-    )
-    (property "Datasheet" "~" (id 3) (at 39.37 177.8 0)
-      (effects (font (size 1.27 1.27)) hide)
-    )
-  )
   (symbol (lib_id "Switch:SW_Push") (at 255.27 25.4 0) (unit 1)
     (in_bom yes) (on_board yes)
@@
       (reference "H5") (unit 1) (value "MountingHole") (footprint "random-keyboard-parts:M2 Mounting Hole")
     )
-    (path "/e0ffc4a5-acee-444d-9091-cb09a2fd596a"
-      (reference "H6") (unit 1) (value "MountingHole") (footprint "random-keyboard-parts:M2 Mounting Hole")
-    )
-    (path "/10fcbf2d-6552-4910-ae9e-906304f0e093"
-      (reference "H7") (unit 1) (value "MountingHole") (footprint "random-keyboard-parts:M2 Mounting Hole")
-    )
-    (path "/339b77fe-16f3-43b4-8399-7230a8ae2102"
-      (reference "H8") (unit 1) (value "MountingHole") (footprint "random-keyboard-parts:M2 Mounting Hole")
-    )
-    (path "/3427d123-61e2-4c57-80e1-efb5d2751d47"
-      (reference "H9") (unit 1) (value "MountingHole") (footprint "random-keyboard-parts:M2 Mounting Hole")
-    )
     (path "/00000000-0000-0000-0000-000062166a49"
