File: Map/map-plate.kicad_pcb (KiCad board)
At the start: 2 copper layers, 385.8 x 95.3 mm, 7 parts

Commit message: Update List and Map
Update List and Map
Parts:
- removed G2: string_dotlen, Images:map-dotlen108mm
- added H5: MountingHole, random-keyboard-parts:M2 Mounting Hole, F.Cu at (52.5, 98.9)
- added H5: MountingHole, random-keyboard-parts:M2 Mounting Hole, F.Cu at (376.3, -1.11)
- added H5: MountingHole, random-keyboard-parts:M2 Mounting Hole, F.Cu at (376.3, 98.9)
- added H5: MountingHole, random-keyboard-parts:M2 Mounting Hole, F.Cu at (214.4, -1.11)
- added H5: MountingHole, random-keyboard-parts:M2 Mounting Hole, F.Cu at (52.5, -1.11)
- added H5: MountingHole, random-keyboard-parts:M2 Mounting Hole, F.Cu at (214.4, 98.9)
Other:
- board size 385.8 x 95.3 mm -> 385.8 x 104.8 mm
